File: Details.kicad_sch (KiCad schematic)
At the start: 2 parts, among them U1 ESP32-S3-WROOM-1

Commit message: initial commit
Parts:
- removed C4: 10uf, symbol Device:C
- removed U1: ESP32-S3-WROOM-1, PCM_Espressif:ESP32-S3-WROOM-1, symbol PCM_Espressif:ESP32-S3-WROOM-1
- added C1: 22uf, Capacitor_SMD:C_0603_1608Metric_Pad1.08x0.95mm_HandSolder, symbol Device:C
- added C4, C62: TBD, Capacitor_SMD:C_0603_1608Metric_Pad1.08x0.95mm_HandSolder, symbol Device:C_Small
- added C60, C61, C63: 22uf, Capacitor_SMD:C_0603_1608Metric_Pad1.08x0.95mm_HandSolder, symbol Device:C_Small
- added J2: BHeader_Conn_02x20_Counter_Clockwise, Connector_PinSocket_2.54mm:PinSocket_2x15_P2.54mm_Vertical, symbol Connector_Generic:Conn_02x15_Odd_Even
- added J3: USB_C_Receptacle, Connector_USB:USB_C_Receptacle_GCT_USB4110, symbol Connector:USB_C_Receptacle_USB2.0_16P
- added R1, R2: 5.1K, Resistor_SMD:R_0603_1608Metric_Pad0.98x0.95mm_HandSolder, symbol Device:R_Small
- added R23, R24: 2.2K, Resistor_SMD:R_0603_1608Metric_Pad0.98x0.95mm_HandSolder, symbol Device:R_Small_US
- added R4: TBD, Capacitor_SMD:C_0603_1608Metric_Pad1.08x0.95mm_HandSolder, symbol Device:R_Small
- added R40: 10K, Resistor_SMD:R_0603_1608Metric_Pad0.98x0.95mm_HandSolder, symbol Device:R_Small
- added SW2: RST, Button_Switch_SMD:SW_SPST_PTS647_Sx38, symbol Switch:SW_Push
- added U1: usblc6-2, Package_TO_SOT_SMD:SOT-23-6, symbol Power_Protection:USBLC6-2SC6
- added U5: ESP32-S3-WROOM-1, PCM_Espressif:ESP32-S3-WROOM-1U, symbol PCM_Espressif:ESP32-S3-WROOM-1
- added U8: ~, symbol 24_lcd_module:24_lcd_module
Connections:
- net GND: now also C1.1, C4.2, C60.1, C61.1, C62.2, C63.1, J2.1 (Pin_1), J2.3 (Pin_3), J2.5 (Pin_5), J3.A1 (GND), J3.A12 (GND), J3.B1 (GND), J3.B12 (GND), J3.S1 (SHIELD), R1.2, R2.2, SW2.2, U1.2 (GND), U5.1 (GND), U5.40 (GND), U5.41 (GND), U8. (SD_SCK)
- new net: C4.1, R4.2, U8. (SD_SCK)
- new net: J3.A5 (CC1), R1.1
- new net: J3.B5 (CC2), R2.1
- new net +BATT: J2.30 (Pin_30)
- new net AXP_PWROK: C62.1, U5.3 (EN)
- new net BOOT: C63.2, J2.24 (Pin_24), R40.2, SW2.1, U5.27 (GPIO0/BOOT)
- new net BUS_OUT: J2.28 (Pin_28)
- new net CSI_D0: U5.25 (GPIO48/SPICLK_N/SUBSPICLK_N_DIFF)
- new net CSI_D1: U5.38 (GPIO2/TOUCH2/ADC1_CH1)
- new net CSI_D2: U5.34 (MTDI/GPIO41/CLK_OUT1)
- new net CSI_D3: U5.15 (GPIO3/TOUCH3/ADC1_CH2)
- new net CSI_D4: U5.17 (GPIO9/TOUCH9/ADC1_CH8/FSPIHD/SUBSPIHD)
- new net CSI_D5: U5.18 (GPIO10/TOUCH10/ADC1_CH9/FSPICS0/FSPIIO4/SUBSPICS0)
- new net CSI_D6: U5.21 (GPIO13/TOUCH13/ADC2_CH2/FSPIQ/FSPIIO7/SUBSPIQ)
- new net CSI_D7: U5.22 (GPIO14/TOUCH14/ADC2_CH3/FSPIWP/FSPIDQS/SUBSPIWP)
- new net CSI_HSYNC: U5.8 (GPIO15/U0RTS/ADC2_CH4/XTAL_32K_P)
- new net CSI_PCLK: U5.26 (GPIO45)
- new net CSI_VSYNC: U5.16 (GPIO46)
- new net GPIO4: J2.2 (Pin_2), U5.4 (GPIO4/TOUCH4/ADC1_CH3)
- new net GPIO5: J2.4 (Pin_4), U5.5 (GPIO5/TOUCH5/ADC1_CH4)
- new net GPIO6: J2.8 (Pin_8), U5.6 (GPIO6/TOUCH6/ADC1_CH5)
- new net GPIO7: J2.21 (Pin_21), U5.7 (GPIO7/TOUCH7/ADC1_CH6)
- new net GPIO8: J2.22 (Pin_22), U5.12 (GPIO8/TOUCH8/ADC1_CH7/SUBSPICS1)
- new net I2C_SCL: J2.18 (Pin_18), R24.2, U5.20 (GPIO12/TOUCH12/ADC2_CH1/FSPICLK/FSPIIO6/SUBSPICLK)
- new net I2C_SDA: J2.17 (Pin_17), R23.2, U5.19 (GPIO11/TOUCH11/ADC2_CH0/FSPID/FSPIIO5/SUBSPID)
- new net INTERUPT_TOUCH: U5.39 (GPIO1/TOUCH1/ADC1_CH0), U8. (SD_SCK)
- new net LCD_CS: U5.9 (GPIO16/U0CTS/ADC2_CH5/XTAL_32K_N), U8. (SD_SCK)
- new net LCD_DC: U5.32 (MTCK/GPIO39/CLK_OUT3/SUBSPICS1), U8. (SD_SCK)
- new net LCD_VDD: R4.1, U8. (SD_SCK)
- new net MCU_EN: J2.6 (Pin_6)
- new net MCU_VDD: C60.2, C61.2, J2.12 (Pin_12), R23.1, R24.1, R40.1, U5.2 (3V3)
- new net SD_CARD_CS: U5.35 (MTMS/GPIO42), U8. (SD_SCK)
- new net SPI_MISO: J2.9 (Pin_9), U5.24 (GPIO47/SPICLK_P/SUBSPICLK_P_DIFF), U8. (SD_SCK)
- new net SPI_MOSI: J2.7 (Pin_7), U5.31 (GPIO38/FSPIWP/SUBSPIWP), U8. (SD_SCK)
- new net SPI_SCK: J2.11 (Pin_11), U5.23 (GPIO21), U8. (SD_SCK)
- new net TOUCH_CS: U5.33 (MTDO/GPIO40/CLK_OUT2), U8. (SD_SCK)
- new net U1RXD: J2.15 (Pin_15), U5.11 (GPIO18/U1RXD/ADC2_CH7/CLK_OUT3)
- new net U1TXD: J2.16 (Pin_16), U5.10 (GPIO17/U1TXD/ADC2_CH6)
- new net UORXD: J2.13 (Pin_13), U5.36 (U0RXD/GPIO44/CLK_OUT2)
- new net UOTXD: J2.14 (Pin_14), U5.37 (U0TXD/GPIO43/CLK_OUT1)
- new net USB_P_N: J3.A7 (D-), J3.B7 (D-), U1.1 (I/O1)
- new net USB_P_P: J3.A6 (D+), J3.B6 (D+), U1.3 (I/O2)
- new net USB_S_N: U1.6 (I/O1), U5.13 (GPIO19/U1RTS/ADC2_CH8/CLK_OUT2/USB_D-)
- new net USB_S_P: U1.4 (I/O2), U5.14 (GPIO20/U1CTS/ADC2_CH9/CLK_OUT1/USB_D+)
- new net VUSB: C1.2, J3.A4 (VBUS), J3.A9 (VBUS), J3.B4 (VBUS), J3.B9 (VBUS), U1.5 (VBUS)
- no-connect marks 0 -> 14
Other:
- company: (none) -> Buildybee
- title: (none) -> BEEPRO
