File: beePro.kicad_pcb (KiCad board)
At the start: 2 copper layers, 1 part

Commit message: initial commit
Parts:
- removed IC**: BMI323, imu:BMI323
- added C1: 22uf, Capacitor_SMD:C_0603_1608Metric_Pad1.08x0.95mm_HandSolder, B.Cu at (112.1, 84.4)
- added C11: 4.7uf, Capacitor_SMD:C_0603_1608Metric_Pad1.08x0.95mm_HandSolder, B.Cu at (120.9, 73.5)
- added C12: 4.7uf, Capacitor_SMD:C_0603_1608Metric_Pad1.08x0.95mm_HandSolder, B.Cu at (133.7, 73.1)
- added C13: 10uf, Capacitor_SMD:C_0603_1608Metric_Pad1.08x0.95mm_HandSolder, F.Cu at (143.5, 53.5)
- added C14: 100nf, Capacitor_SMD:C_0603_1608Metric_Pad1.08x0.95mm_HandSolder, F.Cu at (142.0, 53.5)
- added C15: ????, Capacitor_SMD:C_0603_1608Metric_Pad1.08x0.95mm_HandSolder, F.Cu at (129.9, 83.7)
- added C16: 15pf, Capacitor_SMD:C_0603_1608Metric_Pad1.08x0.95mm_HandSolder, F.Cu at (122.5, 83.9)
- added C17: 10uf, Capacitor_SMD:C_0603_1608Metric_Pad1.08x0.95mm_HandSolder, B.Cu at (138.3, 73.7)
- added C18: 100nf, Capacitor_SMD:C_0603_1608Metric_Pad1.08x0.95mm_HandSolder, F.Cu at (140.8, 80.7)
- added C2: 22uf, Capacitor_SMD:C_0603_1608Metric_Pad1.08x0.95mm_HandSolder, B.Cu at (131.8, 52.2)
- added C20: 100nf, Capacitor_SMD:C_0603_1608Metric_Pad1.08x0.95mm_HandSolder, F.Cu at (142.7, 59.1)
- added C21: 220nf, Capacitor_SMD:C_0603_1608Metric_Pad1.08x0.95mm_HandSolder, F.Cu at (143.8, 61.7)
- added C22: 100nf, Capacitor_SMD:C_0603_1608Metric_Pad1.08x0.95mm_HandSolder, F.Cu at (111.6, 61.9)
- added C23: 10uf, Capacitor_SMD:C_0603_1608Metric_Pad1.08x0.95mm_HandSolder, F.Cu at (120.8, 78.9)
- added C24: 470nf, Capacitor_SMD:C_0603_1608Metric_Pad1.08x0.95mm_HandSolder, F.Cu at (120.8, 80.4)
- added C25: ????, Capacitor_SMD:C_0603_1608Metric_Pad1.08x0.95mm_HandSolder, F.Cu at (129.9, 87.8)
- added C26: 0.1uf, Capacitor_SMD:C_0603_1608Metric_Pad1.08x0.95mm_HandSolder, F.Cu at (133.3, 87.8)
- added C27: 10uf, Capacitor_SMD:C_0603_1608Metric_Pad1.08x0.95mm_HandSolder, F.Cu at (113.7, 69.2)
- added C29: 4.7uf, Capacitor_SMD:C_0603_1608Metric_Pad1.08x0.95mm_HandSolder, B.Cu at (135.2, 73.1)
- added C3: 22uf, Capacitor_SMD:C_0603_1608Metric_Pad1.08x0.95mm_HandSolder, B.Cu at (123.1, 68.5)
- added C30: 22uf, Capacitor_SMD:C_0603_1608Metric_Pad1.08x0.95mm_HandSolder, B.Cu at (131.7, 53.7)
- added C31: 22uf, Capacitor_SMD:C_0603_1608Metric_Pad1.08x0.95mm_HandSolder, B.Cu at (118.3, 62.1)
- added C32: 1uf, Capacitor_SMD:C_0603_1608Metric_Pad1.08x0.95mm_HandSolder, B.Cu at (128.2, 75.7)
- added C33: 0.22uf, Capacitor_SMD:C_0603_1608Metric_Pad1.08x0.95mm_HandSolder, B.Cu at (132.5, 84.0)
- added C34: 1uf, Capacitor_SMD:C_0603_1608Metric_Pad1.08x0.95mm_HandSolder, B.Cu at (128.2, 77.2)
- added C35: 1uf, Capacitor_SMD:C_0603_1608Metric_Pad1.08x0.95mm_HandSolder, B.Cu at (128.2, 81.7)
- added C36: 100pf, Capacitor_SMD:C_0603_1608Metric_Pad1.08x0.95mm_HandSolder, B.Cu at (128.2, 78.7)
- added C37: 10uf, Capacitor_SMD:C_0603_1608Metric_Pad1.08x0.95mm_HandSolder, B.Cu at (124.6, 77.3)
- added C38: 1nf, Capacitor_SMD:C_0603_1608Metric_Pad1.08x0.95mm_HandSolder, B.Cu at (140.8, 88.2)
- added C39: 1uf, Capacitor_SMD:C_0603_1608Metric_Pad1.08x0.95mm_HandSolder, B.Cu at (117.4, 71.8)
- added C40: 1uf, Capacitor_SMD:C_0603_1608Metric_Pad1.08x0.95mm_HandSolder, B.Cu at (117.4, 73.5)
- added C41: 10uf, Capacitor_SMD:C_0603_1608Metric_Pad1.08x0.95mm_HandSolder, B.Cu at (142.4, 88.2)
- added C42: 4.7uf, Capacitor_SMD:C_0603_1608Metric_Pad1.08x0.95mm_HandSolder, B.Cu at (128.2, 74.1)
- added C43: 10uf, Capacitor_SMD:C_0603_1608Metric_Pad1.08x0.95mm_HandSolder, B.Cu at (141.1, 71.0)
- added C44: 10uf, Capacitor_SMD:C_0603_1608Metric_Pad1.08x0.95mm_HandSolder, B.Cu at (138.9, 84.0)
- added C45: 4.7uf, Capacitor_SMD:C_0603_1608Metric_Pad1.08x0.95mm_HandSolder, B.Cu at (120.8, 71.8)
- added C47: 1uf, Capacitor_SMD:C_0603_1608Metric_Pad1.08x0.95mm_HandSolder, B.Cu at (132.2, 73.1)
- added C48: 22uf, Capacitor_SMD:C_0603_1608Metric_Pad1.08x0.95mm_HandSolder, B.Cu at (112.8, 69.5)
- added C49: 22uf, Capacitor_SMD:C_0603_1608Metric_Pad1.08x0.95mm_HandSolder, B.Cu at (118.4, 65.5)
- added C5: 15pf, Capacitor_SMD:C_0603_1608Metric_Pad1.08x0.95mm_HandSolder, F.Cu at (120.7, 73.7)
- added C50: 1nf, Capacitor_SMD:C_0603_1608Metric_Pad1.08x0.95mm_HandSolder, B.Cu at (141.2, 72.8)
- added C51: 10uf, Capacitor_SMD:C_0603_1608Metric_Pad1.08x0.95mm_HandSolder, B.Cu at (138.4, 77.3)
- added C52: 10uf, Capacitor_SMD:C_0603_1608Metric_Pad1.08x0.95mm_HandSolder, B.Cu at (138.4, 80.7)
- added C53: 1uf, Capacitor_SMD:C_0603_1608Metric_Pad1.08x0.95mm_HandSolder, B.Cu at (118.4, 63.7)
- added C54: 1uf, Capacitor_SMD:C_0603_1608Metric_Pad1.08x0.95mm_HandSolder, B.Cu at (130.7, 73.1)
- added C55: 1uf, Capacitor_SMD:C_0603_1608Metric_Pad1.08x0.95mm_HandSolder, B.Cu at (131.8, 56.9)
- added C56: 1uf, Capacitor_SMD:C_0603_1608Metric_Pad1.08x0.95mm_HandSolder, B.Cu at (114.1, 80.8)
- added C57: 1uf, Capacitor_SMD:C_0603_1608Metric_Pad1.08x0.95mm_HandSolder, B.Cu at (126.0, 67.6)
- added C58: 1uf, Capacitor_SMD:C_0603_1608Metric_Pad1.08x0.95mm_HandSolder, B.Cu at (120.8, 76.7)
- added C59: 1nf, Capacitor_SMD:C_0603_1608Metric_Pad1.08x0.95mm_HandSolder, B.Cu at (137.2, 84.0)
- added C6: 22uf, Capacitor_SMD:C_0603_1608Metric_Pad1.08x0.95mm_HandSolder, B.Cu at (112.8, 71.3)
- added C60: 22uf, Capacitor_SMD:C_0603_1608Metric_Pad1.08x0.95mm_HandSolder, F.Cu at (114.5, 51.8)
- added C61: 22uf, Capacitor_SMD:C_0603_1608Metric_Pad1.08x0.95mm_HandSolder, F.Cu at (114.5, 53.4)
- added C62: TBD, Capacitor_SMD:C_0603_1608Metric_Pad1.08x0.95mm_HandSolder, F.Cu at (114.7, 58.4)
- added C63: 22uf, Capacitor_SMD:C_0603_1608Metric_Pad1.08x0.95mm_HandSolder, B.Cu at (123.3, 56.8)
- added C64: 100nf, Capacitor_SMD:C_0603_1608Metric_Pad1.08x0.95mm_HandSolder, F.Cu at (127.0, 77.4)
- added C65: 100nf, Capacitor_SMD:C_0603_1608Metric_Pad1.08x0.95mm_HandSolder, F.Cu at (128.5, 77.4)
- added C7: 22uf, Capacitor_SMD:C_0603_1608Metric_Pad1.08x0.95mm_HandSolder, B.Cu at (112.7, 67.9)
- added C72: .1uf, Capacitor_SMD:C_0603_1608Metric_Pad1.08x0.95mm_HandSolder, B.Cu at (124.5, 75.7)
- added C73: 4.7uf, Capacitor_SMD:C_0603_1608Metric_Pad1.08x0.95mm_HandSolder, B.Cu at (121.9, 81.4)
- added C8: 220uf/6.3V, Capacitor_SMD:CP_Elec_6.3x5.3, B.Cu at (137.9, 66.2)
- added C9: 220uf/6.3V, Capacitor_SMD:CP_Elec_6.3x5.3, B.Cu at (125.1, 62.4)
- added D2: CHRG, LED_SMD:LED_0603_1608Metric_Pad1.05x0.95mm_HandSolder, B.Cu at (124.5, 72.7)
- added D6: 5.1V, Diode_SMD:D_SOD-123, B.Cu at (112.9, 73.8)
- added D8: SS24, Diode_SMD:D_SMA, B.Cu at (114.2, 59.0)
- added IC2: AXP192, AXP192:QFN40P600X600X92-49N-D, B.Cu at (133.7, 78.5)
- added J1: Cam_Conn_01x24_MountingPin, Connector_FFC-FPC:Hirose_FH12-24S-0.5SH_1x24-1MP_P0.50mm_Horizontal, F.Cu at (115.8, 80.9)
- added J2: BHeader_Conn_02x20_Counter_Clockwise, Connector_PinSocket_2.54mm:PinSocket_2x15_P2.54mm_Vertical, B.Cu at (145.6, 52.3)
- added J3: USB_C_Receptacle, Connector_USB:USB_C_Receptacle_GCT_USB4110, B.Cu at (122.3, 87.4)
- added J4: Battery connector, Connector_JST:JST_PH_B2B-PH-K_1x02_P2.00mm_Vertical, B.Cu at (139.7, 53.7)
- added L1: 2.2uH, Inductor_SMD:L_Cenker_CKCS252012, B.Cu at (137.6, 87.9)
- added L2: 2.2uH, Inductor_SMD:L_Cenker_CKCS252012, B.Cu at (133.4, 88.0)
- added L3: 4.7uH, Inductor_SMD:L_Changjiang_FNR5012S, B.Cu at (113.4, 64.1)
- added L4: 4.7uH, Inductor_SMD:L_Cenker_CKCS252012, B.Cu at (141.4, 84.1)
- added R1: 5.1K, Resistor_SMD:R_0603_1608Metric_Pad0.98x0.95mm_HandSolder, B.Cu at (112.7, 81.0)
- added R10: 10K, Resistor_SMD:R_0603_1608Metric_Pad0.98x0.95mm_HandSolder, F.Cu at (129.2, 71.7)
- added R11: 2.2ohm, Resistor_SMD:R_0603_1608Metric_Pad0.98x0.95mm_HandSolder, B.Cu at (120.8, 75.1)
- added R12: 10K, Resistor_SMD:R_0603_1608Metric_Pad0.98x0.95mm_HandSolder, B.Cu at (135.7, 84.0)
- added R13: 200K, Resistor_SMD:R_0603_1608Metric_Pad0.98x0.95mm_HandSolder, B.Cu at (128.2, 80.2)
- added R14: 10K, Resistor_SMD:R_0603_1608Metric_Pad0.98x0.95mm_HandSolder, B.Cu at (131.0, 84.0)
- added R15: 7.33R16, Resistor_SMD:R_0603_1608Metric_Pad0.98x0.95mm_HandSolder, B.Cu at (120.1, 68.4)
- added R16: 5K, Resistor_SMD:R_0603_1608Metric_Pad0.98x0.95mm_HandSolder, B.Cu at (121.6, 68.5)
- added R17: 10K, Resistor_SMD:R_0603_1608Metric_Pad0.98x0.95mm_HandSolder, B.Cu at (111.2, 53.2)
- added R18: 2k2, Resistor_SMD:R_0603_1608Metric_Pad0.98x0.95mm_HandSolder, F.Cu at (137.9, 84.1)
- added R2: 5.1K, Resistor_SMD:R_0603_1608Metric_Pad0.98x0.95mm_HandSolder, B.Cu at (113.7, 84.4)
- added R20: ???, Resistor_SMD:R_0603_1608Metric_Pad0.98x0.95mm_HandSolder, B.Cu at (131.7, 55.3)
- added R23: 2.2K, Resistor_SMD:R_0603_1608Metric_Pad0.98x0.95mm_HandSolder, F.Cu at (115.3, 65.6)
- added R24: 2.2K, Resistor_SMD:R_0603_1608Metric_Pad0.98x0.95mm_HandSolder, F.Cu at (113.5, 61.7)
- added R25: 1, Resistor_SMD:R_2512_6332Metric, B.Cu at (141.2, 78.1)
- added R27: 10K, Resistor_SMD:R_0603_1608Metric_Pad0.98x0.95mm_HandSolder, B.Cu at (134.0, 84.0)
- added R3: 4K7, Resistor_SMD:R_0603_1608Metric_Pad0.98x0.95mm_HandSolder, B.Cu at (117.1, 75.4)
- added R30: 470, Resistor_SMD:R_0603_1608Metric_Pad0.98x0.95mm_HandSolder, B.Cu at (124.6, 74.1)
- added R31: 10K, Resistor_SMD:R_0603_1608Metric_Pad0.98x0.95mm_HandSolder, B.Cu at (136.8, 73.1)
- added R32: 10K, Resistor_SMD:R_0603_1608Metric_Pad0.98x0.95mm_HandSolder, B.Cu at (128.9, 69.1)
- added R33: ???, Resistor_SMD:R_0603_1608Metric_Pad0.98x0.95mm_HandSolder, B.Cu at (131.8, 62.1)
- added R34: 10K, Resistor_SMD:R_0603_1608Metric_Pad0.98x0.95mm_HandSolder, B.Cu at (128.1, 72.4)
- added R35: ???, Resistor_SMD:R_0603_1608Metric_Pad0.98x0.95mm_HandSolder, B.Cu at (132.2, 69.2)
- added R36: 10K, Resistor_SMD:R_0603_1608Metric_Pad0.98x0.95mm_HandSolder, B.Cu at (111.1, 81.0)
- added R37: TBD, Capacitor_SMD:C_0603_1608Metric_Pad1.08x0.95mm_HandSolder, F.Cu at (114.7, 55.9)
- added R38: 10K, Resistor_SMD:R_0603_1608Metric_Pad0.98x0.95mm_HandSolder, F.Cu at (113.7, 65.7)
- added R40: 10K, Resistor_SMD:R_0603_1608Metric_Pad0.98x0.95mm_HandSolder, B.Cu at (126.8, 56.8)
- added R5: 10K, Resistor_SMD:R_0603_1608Metric_Pad0.98x0.95mm_HandSolder, F.Cu at (140.5, 63.9)
- added R6: 10K, Resistor_SMD:R_0603_1608Metric_Pad0.98x0.95mm_HandSolder, B.Cu at (117.1, 76.9)
- added R8: 1k, Resistor_SMD:R_0603_1608Metric_Pad0.98x0.95mm_HandSolder, F.Cu at (120.9, 83.9)
- added R9: 10K, Resistor_SMD:R_0603_1608Metric_Pad0.98x0.95mm_HandSolder, F.Cu at (132.4, 82.8)
- added SW1: PWR, Button_Switch_SMD:SW_SPST_PTS647_Sx38, B.Cu at (116.3, 53.1)
- added SW2: RST, Button_Switch_SMD:SW_SPST_PTS647_Sx38, B.Cu at (125.3, 53.1)
- added U1: usblc6-2, Package_TO_SOT_SMD:SOT-23-6, B.Cu at (112.4, 87.8)
- added U10: VEML7700, VEML7700-TR:XDCR_VEML7700-TR, F.Cu at (111.2, 67.4)
- added U11: MT3608, Package_TO_SOT_SMD:SOT-23-6, B.Cu at (116.9, 68.6)
- added U12: LSM6DS3, Package_LGA:LGA-14_3x2.5mm_P0.5mm_LayoutBorder3x4y, F.Cu at (127.4, 74.0)
- added U13: MIC5504-2.8YM5, Package_TO_SOT_SMD:SOT-23-5, B.Cu at (112.3, 76.8)
- added U14: PCA9536D, Package_SO:SOIC-8_3.9x4.9mm_P1.27mm, F.Cu at (133.7, 75.3)
- added U2: NCP380HMU05AATBG, NCP380HMU05AATBG:UDFN6_2X2_ONS, B.Cu at (131.8, 59.4)
- added U3: LIS2MDL, Package_LGA:LGA-12_2x2mm_P0.5mm, F.Cu at (141.4, 61.3)
- added U4: MCP7940N-xMNY, Package_DFN_QFN:DFN-8-1EP_3x2mm_P0.5mm_EP1.36x1.46mm, F.Cu at (130.5, 85.7)
- added U5: ESP32-S3-WROOM-1, PCM_Espressif:ESP32-S3-WROOM-1U, F.Cu at (127.3, 59.8)
- added U6: AHT20, aht20:AHT20, F.Cu at (137.5, 80.7)
- added U7: NCP380HMU05AATBG, NCP380HMU05AATBG:UDFN6_2X2_ONS, B.Cu at (131.6, 64.5)
- added U9: NCP380HMU05AATBG, NCP380HMU05AATBG:UDFN6_2X2_ONS, B.Cu at (126.0, 70.1)
- added X1: 20MHz, Oscillator:Oscillator_SMD_Abracon_ASE-4Pin_3.2x2.5mm, F.Cu at (121.0, 76.3)
- added Y1: 32.768kHz, Crystal:Crystal_SMD_3215-2Pin_3.2x1.5mm, F.Cu at (127.1, 85.7)
Other:
- board outline added: 40 x 40 mm
- copper layers 2 -> 4
