File: beePro.kicad_sch (KiCad schematic)
At the start: 10 parts, among them J1 SD_Card, U1 ESP32-S3-WROOM-1, U2 AMS1117-3.3, U3 MPU-6050, U4 INA226

Commit message: inital commit
Parts:
- removed C1, C2, C4, C5: C, symbol Device:C
- removed C3: C_Polarized, symbol Device:C_Polarized
- removed J1: SD_Card, symbol Connector:SD_Card
- removed U1: ESP32-S3-WROOM-1, PCM_Espressif:ESP32-S3-WROOM-1, symbol PCM_Espressif:ESP32-S3-WROOM-1
- removed U2: AMS1117-3.3, Package_TO_SOT_SMD:SOT-223-3_TabPin2, symbol Regulator_Linear:AMS1117-3.3
- removed U3: MPU-6050, Sensor_Motion:InvenSense_QFN-24_4x4mm_P0.5mm, symbol Sensor_Motion:MPU-6050
- removed U4: INA226, Package_SO:VSSOP-10_3x3mm_P0.5mm, symbol Sensor_Energy:INA226
Connections:
- no-connect marks 0 -> 2
Other:
- added sheet esp32 (Details.kicad_sch)
- added sheet i2s_amp-spi_lcd_sdcard (spi_lcd_sdcard.kicad_sch)
- added sheet ports (ports.kicad_sch)
- added sheet pwr_mgmt (pwr_mgmt.kicad_sch)
- added sheet sensors (esp32s3.kicad_sch)
- note added: "https://www.espressif.com/sites/default/files/documentation/esp32-s3_datasheet_en.pdf"
- note added: "https://www.ti.com/lit/ds/symlink/tps73633-ep.pdf?ts=1716467232035&ref_url=https%253A%252F%252Fwww.google.com%252F"

Commit message: initial commit
Connections:
- no-connect marks 2 -> 0
Other:
- sheet esp32 renamed mcu
- sheet i2s_amp-spi_lcd_sdcard renamed peripherals
- removed sheet ports
- note added: "NOT USING IN V1.0"
- note removed: "https://www.espressif.com/sites/default/files/documentation/esp32-s3_datasheet_en.pdf"
- note removed: "https://www.ti.com/lit/ds/symlink/tps73633-ep.pdf?ts=1716467232035&ref_url=https%253A%252F%252Fwww.google.com%252F"
- company: (none) -> Buildybee
- title: (none) -> BEEPRO
