File: esp32s3.kicad_sch (KiCad schematic)
At the start: 23 parts, among them IC1 HMC5883L, U10 VCNL4040M3OE, U3 MPU-6050, U4 MCP7940N-xMNY, U6 AHT20, Y1 32.768kHz

Commit message: initial commit
Parts:
- removed BT1: HOW???, symbol Device:Battery_Cell
- removed C13, C14, C15, C20, C27: 0.1uf, symbol Device:C
- removed C21: 2.2nf, symbol Device:C
- removed C22: 10nf, symbol Device:C
- removed C23: 4.7uf, symbol Device:C
- removed C24: 0.22uf, symbol Device:C
- removed C25, C26: ????, symbol Device:C
- removed C28: 2.2uf, symbol Device:C
- removed IC1: HMC5883L, HMC5883L, symbol HMC5883L:HMC5883L
- removed R10: 8.2K, symbol Device:R
- removed R5: 4k7, symbol Device:R
- removed R9: 10K, symbol Device:R
- removed U3: MPU-6050, Sensor_Motion:InvenSense_QFN-24_4x4mm_P0.5mm, symbol Sensor_Motion:MPU-6050
- removed U4: MCP7940N-xMNY, Package_DFN_QFN:DFN-8-1EP_3x2mm_P0.5mm_EP1.36x1.46mm, symbol Timer_RTC:MCP7940N-xMNY
- removed Y1: 32.768kHz, symbol Device:Crystal
- added C13, C23, C27: 10uf, Capacitor_SMD:C_0603_1608Metric_Pad1.08x0.95mm_HandSolder, symbol Device:C_Small
- added C14, C20, C22, C64, C65: 100nf, Capacitor_SMD:C_0603_1608Metric_Pad1.08x0.95mm_HandSolder, symbol Device:C_Small
- added C16, C5: 15pf, Capacitor_SMD:C_0603_1608Metric_Pad1.08x0.95mm_HandSolder, symbol Device:C_Small
- added C21: 220nf, Capacitor_SMD:C_0603_1608Metric_Pad1.08x0.95mm_HandSolder, symbol Device:C_Small
- added C24: 470nf, Capacitor_SMD:C_0603_1608Metric_Pad1.08x0.95mm_HandSolder, symbol Device:C_Small
- added J1: Cam_Conn_01x24_MountingPin, Connector_FFC-FPC:Hirose_FH12-24S-0.5SH_1x24-1MP_P0.50mm_Horizontal, symbol Connector_Generic_MountingPin:Conn_01x24_MountingPin
- added R10, R38, R5: 10K, Resistor_SMD:R_0603_1608Metric_Pad0.98x0.95mm_HandSolder, symbol Device:R_Small
- added R8: 1k, Resistor_SMD:R_0603_1608Metric_Pad0.98x0.95mm_HandSolder, symbol Device:R_Small_US
- added U12: LSM6DS3, Package_LGA:LGA-14_3x2.5mm_P0.5mm_LayoutBorder3x4y, symbol Sensor_Motion:LSM6DS3
- added U3: LIS2MDL, Package_LGA:LGA-12_2x2mm_P0.5mm, symbol Sensor_Magnetic:LIS2MDL
- added X1: 20MHz, Oscillator:Oscillator_SMD_Abracon_ASE-4Pin_3.2x2.5mm, symbol Oscillator:ASE-xxxMHz
- C18: footprint (none) -> Capacitor_SMD:C_0603_1608Metric_Pad1.08x0.95mm_HandSolder
- U10: value VCNL4040M3OE -> VEML7700; footprint VCNL4040M3OE:VISHAY_VCNL4040_4X2X1.1 -> VEML7700-TR:XDCR_VEML7700-TR; symbol VCNL4040M3OE:VCNL4040M3OE -> VEML7700-TR:VEML7700-TR; Check_prices https://www.snapeda.com/parts/VCNL4040M3OE/Vishay+Semicondu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 -> https://www.snapeda.com/parts/VEML7700-TR/Vishay+Semiconduc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; Description_1 Optical Sensor Ambient 550nm I2C 8-SMD Module -> Optical Sensor Ambient 545nm I2C 4-SMD, J-Lead; MANUFACTURER (none) -> Vishay; MAXIMUM_PACKAGE_HEIGHT (none) -> 3 mm; MP VCNL4040M3OE -> VEML7700-TR; PARTREV (none) -> 1.6; Package None -> Package; Purchase-URL (none) -> https://www.snapeda.com/api/url_track_click_mouser/?unipart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; SNAPEDA_PN (none) -> VEML7700-TR; STANDARD (none) -> Manufacturer Recommendations; SnapEDA_Link https://www.snapeda.com/parts/VCNL4040M3OE/Vishay+Semicondu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 -> https://www.snapeda.com/parts/VEML7700-TR/Vishay+Semiconduc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
- U6: footprint AHT20 -> aht20:AHT20
Connections:
- net GND: now also U10.3 (GND), C13.1, C14.1, C16.1, C20.1, C21.2, C22.1, C23.2, C24.2, C27.1, C5.1, C64.1, C65.1, J1.10 (Pin_10), J1.23 (Pin_23), J1.MP (MountPin), R8.1, U12.1 (SDO/SA0), U12.2 (SDX), U12.3 (SCX), U12.6 (GND), U12.7 (GND), U3.6 (GND), U3.8 (GND), X1.2 (GND); no longer U10.1
- net +3.3V renamed SENSOR_VDD
- net SENSOR_VDD: now also C13.2, C14.2, C65.2, R10.1, R38.2, R5.2, U12.8 (VDD), U3.9 (Vdd); no longer U10.3, U10.4
- net i2c_sys_scl renamed I2C_SCL
- net I2C_SCL: now also U10.1 (SCL), J1.20 (Pin_20), U12.13 (SCL), U3.1 (SCL/SPC); no longer U10.8
- net i2c_sys_sda renamed I2C_SDA
- net I2C_SDA: now also U10.4 (SDA), J1.22 (Pin_22), U12.14 (SDA), U3.4 (SDA/SDI/SDO); no longer U10.7
- net proximity_cathode: no longer names the net of U10.2 (VDD)
- net proximity_cathode: now also C22.2, C27.2, R38.1; no longer U10.5
- new net: J1.17 (Pin_17), R8.2
- new net: R5.1, U3.3 (~{CS})
- new net: C21.1, U3.5 (C1)
- new net: R10.2, U12.12 (CS)
- new net 1V2_VDD: J1.15 (Pin_15)
- new net 2V8_VDD: C23.1, C24.1, J1.21 (Pin_21), X1.4 (Vdd)
- new net CAM_DOVDD: C16.2, J1.14 (Pin_14)
- new net CAM_RST: J1.19 (Pin_19)
- new net CSI_D0: J1.6 (Pin_6)
- new net CSI_D1: J1.4 (Pin_4)
- new net CSI_D2: J1.3 (Pin_3)
- new net CSI_D3: J1.5 (Pin_5)
- new net CSI_D4: J1.7 (Pin_7)
- new net CSI_D5: J1.9 (Pin_9)
- new net CSI_D6: J1.11 (Pin_11)
- new net CSI_D7: J1.13 (Pin_13)
- new net CSI_HSYNC: J1.16 (Pin_16)
- new net CSI_MCLK: J1.12 (Pin_12), X1.3 (OUT)
- new net CSI_PCLK: C5.2, J1.8 (Pin_8)
- new net CSI_VSYNC: J1.18 (Pin_18)
- new net MCU_VDD: C20.2, C64.2, U12.5 (VDDIO), U3.10 (Vdd_IO)
- no-connect marks 0 -> 9
Other:
- note added: "I2C ADDR : 0x6A"
- note added: "V:2.5 - 3.6v"
- note removed: "I2C ADDR : 0x38"
- note removed: "I2C ADDR : 0x68"
- note removed: "I2C ADDR : 0x6F"
- company: (none) -> Buildybee
- title: (none) -> BEEPRO
- moved on the sheet: C18, U6
