File: ports.kicad_sch (KiCad schematic)
At the start: 13 parts, among them J1 Cam_Conn_01x24_MountingPin, J2 USB_C_Receptacle, J3 BHeader_Conn_02x20_Counter_Cl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, J5 Conn_01x04_Pin, J6 Conn_01x04_Pin, U2 SRV05-4, X1 ASCO

Commit message: initial commit
Parts:
- removed C1: 22uf, symbol Device:C
- removed C17, C5: 15pf, symbol Device:C
- removed J1: Cam_Conn_01x24_MountingPin, symbol Connector_Generic_MountingPin:Conn_01x24_MountingPin
- removed J2: USB_C_Receptacle, Connector_USB:USB_C_Receptacle_Amphenol_12401548E4-2A, symbol Connector:USB_C_Receptacle
- removed J3: BHeader_Conn_02x20_Counter_Clockwise, Connector_Harwin:Harwin_M20-7811545_2x15_P2.54mm_Vertical, symbol Connector_Generic:Conn_02x20_Counter_Clockwise
- removed J5, J6: Conn_01x04_Pin, Connector_JST:JST_EH_S4B-EH_1x04_P2.50mm_Horizontal, symbol Connector:Conn_01x04_Pin
- removed R1, R2: 5.1K, symbol Device:R
- removed R8: 1k, symbol Device:R
- removed U2: SRV05-4, Package_TO_SOT_SMD:SOT-23-6, symbol Power_Protection:SRV05-4
- removed X1: ASCO, Oscillator:Oscillator_SMD_Abracon_ASCO-4Pin_1.6x1.2mm, symbol Oscillator:ASCO
Connections:
- no-connect marks 3 -> 0
