File: pwr_mgmt.kicad_sch (KiCad schematic)
At the start: 43 parts, among them IC2 AXP192, J4 Conn_01x02_Socket, U11 MT3608

Commit message: initial commit
Parts:
- removed C10: 4.7uf, symbol Device:C
- removed C31: 10uf, symbol Device:C
- removed C33: 0.22u, symbol Device:C
- removed C39, C40: 22uf, symbol Device:C
- removed C45, C46: 475uf, symbol Device:C_Polarized_Small_US
- removed D5: D_Schottky, symbol Device:D_Schottky
- removed D7: V ??, symbol Device:D_Schottky
- removed J4: Conn_01x02_Socket, Connector_JST:JST_EH_S2B-EH_1x02_P2.50mm_Horizontal, symbol Connector:Conn_01x02_Socket
- removed R4: 2.2, symbol Device:R
- added C17, C51, C52: 10uf, Capacitor_SMD:C_0603_1608Metric_Pad1.08x0.95mm_HandSolder, symbol Device:C_Small
- added C2, C3, C31, C6, C7: 22uf, Capacitor_SMD:C_0603_1608Metric_Pad1.08x0.95mm_HandSolder, symbol Device:C_Small
- added C33: 0.22uf, Capacitor_SMD:C_0603_1608Metric_Pad1.08x0.95mm_HandSolder, symbol Device:C_Small
- added C39, C40, C53, C54, C55, C56, C57, C58: 1uf, Capacitor_SMD:C_0603_1608Metric_Pad1.08x0.95mm_HandSolder, symbol Device:C_Small
- added C45, C73: 4.7uf, Capacitor_SMD:C_0603_1608Metric_Pad1.08x0.95mm_HandSolder, symbol Device:C_Small
- added C50, C59: 1nf, Capacitor_SMD:C_0603_1608Metric_Pad1.08x0.95mm_HandSolder, symbol Device:C_Small
- added C72: .1uf, Capacitor_SMD:C_0603_1608Metric_Pad1.08x0.95mm_HandSolder, symbol Device:C_Small
- added C8, C9: 220uf/6.3V, Capacitor_SMD:CP_Elec_6.3x5.3, symbol Device:C_Polarized_Small_US
- added D2: CHRG, LED_SMD:LED_0603_1608Metric_Pad1.05x0.95mm_HandSolder, symbol Device:LED_Small_Filled
- added J4: Battery connector, Connector_JST:JST_PH_B2B-PH-K_1x02_P2.00mm_Vertical, symbol Connector:Conn_01x02_Pin
- added L4: 4.7uH, Inductor_SMD:L_Cenker_CKCS252012, symbol Device:L
- added R17, R27, R31, R32, R34, R36: 10K, Resistor_SMD:R_0603_1608Metric_Pad0.98x0.95mm_HandSolder, symbol Device:R_Small_US
- added R20, R33, R35: ???, Resistor_SMD:R_0603_1608Metric_Pad0.98x0.95mm_HandSolder, symbol Device:R_Small_US
- added R25: 1, Resistor_SMD:R_2512_6332Metric, symbol Device:R_Small_US
- added R30: 470, Resistor_SMD:R_0603_1608Metric_Pad0.98x0.95mm_HandSolder, symbol Device:R_Small_US
- added SW1: PWR, Button_Switch_SMD:SW_SPST_PTS647_Sx38, symbol Switch:SW_Push
- added SW3: SW_SPDT, symbol Switch:SW_SPDT
- added U13: MIC5504-2.8YM5, Package_TO_SOT_SMD:SOT-23-5, symbol Regulator_Linear:MIC5504-2.8YM5
- added U2, U7, U9: NCP380HMU05AATBG, NCP380HMU05AATBG:UDFN6_2X2_ONS, symbol NCP380HMU05AATBG:NCP380HMU05AATBG
- C11, C32, C34, C35, C47, C48, C49: footprint (none) -> Capacitor_SMD:C_0603_1608Metric_Pad1.08x0.95mm_HandSolder
- C12, C29, C36, C37, C38: footprint (none) -> Capacitor_SMD:C_0603_1608Metric_Pad1.08x0.95mm_HandSolder; symbol Device:C -> Device:C_Small
- C30: value 4.7uf -> 22uf; footprint (none) -> Capacitor_SMD:C_0603_1608Metric_Pad1.08x0.95mm_HandSolder; symbol Device:C -> Device:C_Small
- C41: value 22uf -> 10uf; footprint (none) -> Capacitor_SMD:C_0603_1608Metric_Pad1.08x0.95mm_HandSolder; symbol Device:C -> Device:C_Small
- C42: value 435uf -> 4.7uf; footprint (none) -> Capacitor_SMD:C_0603_1608Metric_Pad1.08x0.95mm_HandSolder; symbol Device:C_Polarized_Small_US -> Device:C_Small
- C43, C44: value C -> 10uf; footprint (none) -> Capacitor_SMD:C_0603_1608Metric_Pad1.08x0.95mm_HandSolder; symbol Device:C -> Device:C_Small
- D6: value D_Schottky -> 5.1V; footprint (none) -> Diode_SMD:D_SOD-123; symbol Device:D_Schottky -> Device:D_Zener_Small
- D8: value V ?? -> SS24; footprint (none) -> Diode_SMD:D_SMA
- IC2: footprint QFN40P600X600X92-49N-D -> AXP192:QFN40P600X600X92-49N-D
- L1: renamed from 2.2uh; value L -> 2.2uH; footprint (none) -> Inductor_SMD:L_Cenker_CKCS252012
- L2: value uH ?? -> 2.2uH; footprint (none) -> Inductor_SMD:L_Cenker_CKCS252012
- L3: value 47uH ?? -> 4.7uH; footprint (none) -> Inductor_SMD:L_Changjiang_FNR5012S
- R11: value 2.2 -> 2.2ohm; footprint (none) -> Resistor_SMD:R_0603_1608Metric_Pad0.98x0.95mm_HandSolder
- R12, R13, R14: footprint (none) -> Resistor_SMD:R_0603_1608Metric_Pad0.98x0.95mm_HandSolder; symbol Device:R -> Device:R_Small_US
- R15, R16, R3, R6: footprint (none) -> Resistor_SMD:R_0603_1608Metric_Pad0.98x0.95mm_HandSolder
Connections:
- net LDO2 is gone; now on net GND: IC2.11 (LDO3)
- net LDO3 is gone; now on net GND: IC2.12 (LDO2)
- net +BATT: now also C2.1, J4.1 (Pin_1)
- net GND: now also C43.2, IC2.9 (PGND2), C17.1, C2.2, C3.2, C31.2, C33.2, C40.2, C45.1, C45.2, C50.1, C51.1, C52.1, C53.2, C54.2, C55.2, C56.2, C57.2, C58.2, C6.2, C7.2, C72.2, C73.1, C73.2, C8.2, C9.2, J4.2 (Pin_2), R20.2, R32.2, R33.2, R35.2, R36.2, SW1.1, SW3.1 (A), U13.2 (GND), U2.5 (GND), U2.7 (EPAD), U7.5 (GND), U7.7 (EPAD), U9.5 (GND), U9.7 (EPAD); no longer C38.2, C41.2, C43.1, IC2.4 (N_OE)
- net IPS_OUT: now also C43.1, C17.2, C33.1, C39.1, C6.1, C7.1, C8.1, R25.2, R30.1, SW3.3 (C), U13.1 (VIN); no longer C43.2, IC2.13 (LDOIN)
- net PWR_KEY: now also R17.1
- net RTC_VDD: now also C72.1, R27.2
- net VBUS: now also C58.1, U9.1 (OUT)
- net 1V2_VDD: now reaches IC2.10 (DCDC2)
- net 1V2_VDD: now also C50.2, C51.2, L4.2
- net BUS_OUT_EN: now reaches IC2.18 (GPIO1)
- net BUS_OUT_EN: now also R31.1, U2.4 (EN)
- net USB_OUT_EN: now reaches IC2.20 (GPIO2)
- net USB_OUT_EN: now also R32.1, U7.4 (EN)
- net at IC2.27 (PWREN): now also R27.1
- net at IC2.36 (CHGLED): now also D2.1 (K)
- net VUSB_EN: now reaches IC2.41 (GPIO3)
- net VUSB_EN: now also R34.1, U9.4 (EN)
- net CAM_AVDD_EN: now reaches IC2.42 (GPIO4)
- net CAM_AVDD_EN: now also C39.2, R36.1, U13.3 (EN)
- net at IC2.8 (LX2): now also L4.1
- net at R3.2, R6.1, U11.4 (EN): now also C3.1
- net +5V renamed BUS_5V
- net BUS_5V: now also C31.1, C53.1, C54.1, C9.1, R31.2, R34.2, U2.6 (IN), U7.6 (IN)
- net EN_5V_BOOST renamed 5V_BOOST_EN
- net MCU_BSS: no longer names the net of C41.1
- net MCU_BSS: now also C38.2; no longer L1.1
- net MCU_VSS renamed MCU_VDD
- net MCU_VDD: now also C41.2, L1.1
- net PWR1: no longer names the net of C44.2, IC2.17 (DCDC3), L2.1
- net PWR1: now also C59.2
- net USB_5V: no longer names the net of IC2.32 (ACIN_1)
- net USB_5V: no longer IC2.33 (ACIN_2)
- net VBAT_RTC: no longer names the net of IC2.30 (BACKUP)
- net bus_pwr_enable renamed BUS_PWR_EN
- net esp32_reset renamed AXP_PWROK
- net i2c_sys_scl renamed I2C_SCL
- net i2c_sys_sda renamed I2C_SDA
- new net: D2.2 (A), R30.2
- new net: C52.2, IC2.13 (LDOIN), R25.1
- new net: IC2.4 (N_OE), SW3.2 (B)
- new net: R33.1, U7.2 (ILIM)
- new net: R35.1, U9.2 (ILIM)
- new net: R20.1, U2.2 (ILIM)
- new net: R17.2, SW1.2
- new net 2V8_VDD: C40.1, U13.5 (VOUT)
- new net BUS_OUT: C55.1, U2.1 (OUT)
- new net LCD_VDD: C59.1
- new net VUSB: C56.1, C57.1, U7.1 (OUT), U9.6 (IN)
- no-connect marks 8 -> 7
Other:
- note added: "2.8V"
- note added: "5V BOOST -> BUS_OUT(5V IO)"
- note added: "5V BOOST -> USB_OUT(OTG)"
- note added: "5V USB_IN(PWR SOURCE) -> VBUS(AXP_ACIN)"
- note added: "DCDC1 3.3V 1.2A (MCU_VDD) DCDC2 1.2V 1.6A (1V2_VDD) DCDC3 3.3V 0.7A (LCD_VDD)"
- note added: "LDO1 3.3V 30mA (RTC_VDD) LDO2 1.8-3.3V 200mA (SENSOR_VDD) LDO3 1.8-3.3V 200mA (CAM_DOVDD)"
- company: (none) -> Buildybee
- title: (none) -> BEEPRO
- moved on the sheet: C11, C12, C29, C30, C32, C34, C35, C36, C37, C38, C41, C43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
